Commit message: it doesnt work...

File: src/uwu_sim/robots/blobsimp/model.sdf.xacro (robot description, xacro)
@@ -28,24 +28,34 @@
       <xacro:fixed_joint parent="chassis" child="${name}" />
     </xacro:macro>
-    <link name="base_link">
-      <inertial>
-        <mass>0.0001</mass>
-        <inertia>
-          <ixx>1e-09</ixx>
-          <ixy>0</ixy>
-          <ixz>0</ixz>
-          <iyy>1e-09</iyy>
-          <iyz>0</iyz>
-          <izz>1e-09</izz>
-        </inertia>
-      </inertial>
-    </link>
     <include>
       <name>chassis</name>
       <pose relative_to="__model__">0 0 0 0 0 0</pose>
       <uri>model://blobfish_chassis</uri>
+      <!-- <plugin
+        filename="gz-sim-hydrodynamics-system"
+        name="gz::sim::systems::Hydrodynamics">
+        <link_name>chassis</link_name>
+        <xDotU>-4.876161</xDotU>
+        <yDotV>-126.324739</yDotV>
+        <zDotW>-126.324739</zDotW>
+        <kDotP>0</kDotP>
+        <mDotQ>-33.46</mDotQ>
+        <nDotR>-33.46</nDotR>
+        <xUabsU>-6.2282</xUabsU>
+        <xU>0</xU>
+        <yVabsV>-601.27</yVabsV>
+        <yV>0</yV>
+        <zWabsW>-601.27</zWabsW>
+        <zW>0</zW>
+        <kPabsP>-0.1916</kPabsP>
+        <kP>0</kP>
+        <mQabsQ>-632.698957</mQabsQ>
+        <mQ>0</mQ>
+        <nRabsR>-632.698957</nRabsR>
+        <nR>0</nR>
+      </plugin> -->
     </include>
-    <xacro:fixed_joint parent="base_link" child="chassis" />
-    <xacro:thruster name="FL" pose="-0.15 0.18 0 0 0 0" />
+    <xacro:thruster
+      name="FL" pose="-0.15 0.18 0 0 0 0" />
     <xacro:thruster name="ML" pose="-0.15 -0.045 -0.02 -1.5707963267948988 0 0" />
     <xacro:thruster name="BL" pose="-0.15 -0.27 0 -3.141592653589773 0 0" />

Commit message: the simulation is reasonable now. finally.

File: src/uwu_sim/robots/blobsimp/model.sdf.xacro (robot description, xacro)
@@ -6,5 +6,4 @@
         <parent>${parent}</parent>
         <child>${child}</child>
-        <axis />
       </joint>
     </xacro:macro>
@@ -32,30 +31,29 @@
       <pose relative_to="__model__">0 0 0 0 0 0</pose>
       <uri>model://blobfish_chassis</uri>
-      <!-- <plugin
+      <plugin
         filename="gz-sim-hydrodynamics-system"
         name="gz::sim::systems::Hydrodynamics">
-        <link_name>chassis</link_name>
-        <xDotU>-4.876161</xDotU>
-        <yDotV>-126.324739</yDotV>
-        <zDotW>-126.324739</zDotW>
+        <link_name>base_link</link_name>
+        <xDotU>-0.04876161</xDotU>
+        <yDotV>-1.26324739</yDotV>
+        <zDotW>-1.26324739</zDotW>
         <kDotP>0</kDotP>
-        <mDotQ>-33.46</mDotQ>
-        <nDotR>-33.46</nDotR>
-        <xUabsU>-6.2282</xUabsU>
-        <xU>0</xU>
-        <yVabsV>-601.27</yVabsV>
-        <yV>0</yV>
-        <zWabsW>-601.27</zWabsW>
-        <zW>0</zW>
-        <kPabsP>-0.1916</kPabsP>
-        <kP>0</kP>
-        <mQabsQ>-632.698957</mQabsQ>
-        <mQ>0</mQ>
-        <nRabsR>-632.698957</nRabsR>
-        <nR>0</nR>
-      </plugin> -->
+        <mDotQ>-0.3346</mDotQ>
+        <nDotR>-0.3346</nDotR>
+        <xUabsU>-0.62282</xUabsU>
+        <xU>-5</xU>
+        <yVabsV>-60.127</yVabsV>
+        <yV>-5</yV>
+        <zWabsW>-6.0127</zWabsW>
+        <zW>-100</zW>
+        <kPabsP>-0.001916</kPabsP>
+        <kP>-1</kP>
+        <mQabsQ>-6.32698957</mQabsQ>
+        <mQ>-1</mQ>
+        <nRabsR>-6.32698957</nRabsR>
+        <nR>-1</nR>
+      </plugin>
     </include>
-    <xacro:thruster
-      name="FL" pose="-0.15 0.18 0 0 0 0" />
+    <xacro:thruster name="FL" pose="-0.15 0.18 0 0 0 0" />
     <xacro:thruster name="ML" pose="-0.15 -0.045 -0.02 -1.5707963267948988 0 0" />
     <xacro:thruster name="BL" pose="-0.15 -0.27 0 -3.141592653589773 0 0" />

Commit message: merge robot model back into one, part 2

File: src/uwu_sim/robots/blobsimp/model.sdf.xacro (robot description, xacro)
@@ -1,65 +1,25 @@
 <?xml version="1.0"?>
 <sdf version="1.11" xmlns:xacro="http://www.ros.org/wiki/xacro">
+  <xacro:include filename="xacro/chassis.sdf" />
+  <xacro:include filename="xacro/thruster.sdf" />
+  <xacro:macro name="fixed_joint" params="parent child">
+    <joint name="${parent}->${child}_joint" type="fixed">
+      <parent>${parent}</parent>
+      <child>${child}</child>
+    </joint>
+  </xacro:macro>
+  <xacro:macro name="thruster" params="name pose">
+    <xacro:create_thruster name="${name}" pose="${pose}" />
+    <xacro:fixed_joint parent="chassis" child="${name}" />
+  </xacro:macro>
   <model name="blobfish">
-    <xacro:macro name="fixed_joint" params="parent child">
-      <joint name="${child}_joint" type="fixed">
-        <parent>${parent}</parent>
-        <child>${child}</child>
-      </joint>
-    </xacro:macro>
-    <xacro:macro name="thruster" params="name pose">
-      <include>
-        <uri>model://simple_thruster</uri>
-        <name>${name}</name>
-        <pose relative_to="__model__" degrees="true">${pose}</pose>
-        <plugin
-          filename="gz-sim-thruster-system"
-          name="gz::sim::systems::Thruster">
-          <namespace>blobfish/thruster</namespace>
-          <topic>${name}</topic>
-          <joint_name>prop_joint</joint_name>
-          <thrust_coefficient>0.01</thrust_coefficient>
-          <fluid_density>1000</fluid_density>
-          <propeller_diameter>0.076</propeller_diameter>
-        </plugin>
-      </include>
-      <xacro:fixed_joint parent="chassis" child="${name}" />
-    </xacro:macro>
-    <include>
-      <name>chassis</name>
-      <pose relative_to="__model__" degrees="true">0 0 0 0 0 -90</pose>
-      <uri>model://blobfish_chassis</uri>
-      <plugin
-        filename="gz-sim-hydrodynamics-system"
-        name="gz::sim::systems::Hydrodynamics">
-        <link_name>base_link</link_name>
-        <!-- https://gazebosim.org/api/sim/8/theory_hydrodynamics.html -->
-        <xDotU>-0.04876161</xDotU>
-        <yDotV>-1.26324739</yDotV>
-        <zDotW>-1.26324739</zDotW>
-        <kDotP>0</kDotP>
-        <mDotQ>-0.3346</mDotQ>
-        <nDotR>-0.3346</nDotR>
-        <xUabsU>-0.62282</xUabsU>
-        <xU>-5</xU>
-        <yVabsV>-60.127</yVabsV>
-        <yV>-5</yV>
-        <zWabsW>-6.0127</zWabsW>
-        <zW>-100</zW>
-        <kPabsP>-0.001916</kPabsP>
-        <kP>-1</kP>
-        <mQabsQ>-6.32698957</mQabsQ>
-        <mQ>-1</mQ>
-        <nRabsR>-6.32698957</nRabsR>
-        <nR>-1</nR>
-      </plugin>
-    </include>
-    <xacro:thruster name="FL" pose="0.18 0.15 0 0 0 -90" />
-    <xacro:thruster name="FR" pose="0.18 -0.15 0 0 0 -90" />
-    <xacro:thruster name="ML" pose="-0.045 0.15 -0.02 -90 0 0" />
-    <xacro:thruster name="MR" pose="-0.045 -0.15 -0.02 -90 0 0" />
-    <xacro:thruster name="BL" pose="-0.27 0.15 0 0 0 90" />
-    <xacro:thruster name="BR" pose="-0.27 -0.15 0 0 0 90" />
-    <xacro:thruster name="BM" pose="-0.325 0 0.1 -90 0 0" />
+    <xacro:create_chassis name="chassis" />
+    <xacro:thruster name="FL" pose="0.18 0.15 0 0 0 0" />
+    <xacro:thruster name="FR" pose="0.18 -0.15 0 0 0 0" />
+    <xacro:thruster name="ML" pose="-0.045 0.15 0.02 0 -90 0" />
+    <xacro:thruster name="MR" pose="-0.045 -0.15 0.02 0 -90 0" />
+    <xacro:thruster name="BL" pose="-0.27 0.15 0 0 0 180" />
+    <xacro:thruster name="BR" pose="-0.27 -0.15 0 0 0 180" />
+    <xacro:thruster name="BM" pose="-0.325 0 0.13 0 -90 0" />
   </model>
 </sdf>
